File: electronics/TurtleBotController/TurtleBotController/TurtleBotController.kicad_sch (KiCad schematic)
At the start: 10 parts

Commit message: Added lots of files.
Parts:
- added R? (x30): R_.25W_tht, symbol BDK_Passive:R_.25W_tht
- added R? (x2): 1K, Resistor_THT:R_Axial_DIN0207_L6.3mm_D2.5mm_P10.16mm_Horizontal, symbol BDK_Passive:R_.25W_tht
Connections:
- net VCC: now also U?.16 (VCC)
Other:
- moved on the sheet: U?
